File: PCB/air-quality-station.kicad_sch (KiCad schematic)
At the start: 64 parts, among them J1 USB_C_Receptacle_USB2.0_16P, J2 UART, J3 JST_PH_BATTERY, J4 SEN55, J5 I2C_1, J6 I2C_2, J9 E-Paper, Q1 Si1308EDL, U1 ESP32-C6-MINI-1/U, U2 SCD41-D-R2, U3 BMP280, U4 TLV73333PDBV, U5 BQ24075RGT, U6 USBLC6-2P6, U7 TLV73333PDBV, U8 TLV73333PDBV, Y1 32.768kHz

Commit message: Drop battery support, add stitching vias and decooupling capacitors
Parts:
- removed D1: LED, LED_SMD:LED_0603_1608Metric, symbol Device:LED
- removed J3: JST_PH_BATTERY, Connector_JST:JST_PH_B2B-PH-K_1x02_P2.00mm_Vertical, symbol Connector:Conn_01x02_Pin
- removed JP1, JP2: ~, Resistor_SMD:R_0603_1608Metric, symbol Jumper:Jumper_2_Open
- removed R12: 2.2K, Resistor_SMD:R_0603_1608Metric, symbol Device:R
- removed R7, R8, R9: 10K, Resistor_SMD:R_0603_1608Metric, symbol Device:R
- removed U5: BQ24075RGT, Package_DFN_QFN:VQFN-16-1EP_3x3mm_P0.5mm_EP1.6x1.6mm, symbol Battery_Management:BQ24075RGT
- added C28, C29, C30, C31: 100nF, Capacitor_SMD:C_0603_1608Metric, symbol Device:C
- added H3: MountingHole, MountingHole:MountingHole_2.2mm_M2_ISO7380, symbol Mechanical:MountingHole
- added J3: I2C_3, Connector_JST:JST_SH_BM04B-SRSS-TB_1x04-1MP_P1.00mm_Vertical, symbol Connector:Conn_01x04_Pin
- added J7: I2C_4, Connector_JST:JST_SH_BM04B-SRSS-TB_1x04-1MP_P1.00mm_Vertical, symbol Connector:Conn_01x04_Pin
- C6: value 1uF -> 4.7uF; footprint Capacitor_SMD:C_0603_1608Metric -> Capacitor_SMD:C_0805_2012Metric
Connections:
- net +5V_BUS is gone; now on net +5V: C6.1, J1.A4 (VBUS), J1.A9 (VBUS), J1.B4 (VBUS), J1.B9 (VBUS), U6.5 (VBUS)
- net VBAT is gone; now on net +5V: C7.2
- net +3V3_SEN: now also C28.2, C29.1, C30.2, C31.1, J3.2 (Pin_2), J7.2 (Pin_2)
- net +5V: now also C14.1; no longer C14.2
- net GND: now also C14.2, C28.1, C29.2, C30.1, C31.2, J3.1 (Pin_1), J3.MP, J7.1 (Pin_1), J7.MP; no longer C14.1
- net SCL: now also J3.3 (Pin_3), J7.3 (Pin_3)
- net SDA: now also J3.4 (Pin_4), J7.4 (Pin_4)
- no-connect marks 18 -> 16
Other:
- note removed: "Charging circutry"
- moved on the sheet: J2, Q1, R11, R13

Commit message: Improved LDOs, dropped one extension port
Parts:
- removed C31: 100nF, Capacitor_SMD:C_0603_1608Metric, symbol Device:C
- removed J7: I2C_4, Connector_JST:JST_SH_BM04B-SRSS-TB_1x04-1MP_P1.00mm_Vertical, symbol Connector:Conn_01x04_Pin
- removed U4, U7, U8: TLV73333PDBV, Package_TO_SOT_SMD:SOT-23-5, symbol Regulator_Linear:TLV73333PDBV
- added U4, U5, U7: TLV75533PDBV, Package_TO_SOT_SMD:SOT-23-5, symbol Regulator_Linear:TLV75533PDBV
- C4, C5: value 100nF -> 1uF
Connections:
- net +3V3_DISP: now also U7.5 (OUT)
- net +3V3_MCU: now also U5.5 (OUT)
- net +3V3_SEN: now also C30.1, U4.5 (OUT); no longer C30.2
- net +5V: now also U4.1 (IN), U4.3 (EN), U5.1 (IN), U5.3 (EN), U7.1 (IN), U7.3 (EN)
- net GND: now also C30.2, U4.2 (GND), U5.2 (GND), U7.2 (GND); no longer C30.1
Other:
- moved on the sheet: C30
