File: PCB/AHAQ-1.kicad_sch (KiCad schematic)
At the start: 58 parts, among them J1 USB_C_Receptacle_USB2.0_16P, J2 UART, J3 I2C_1, J4 I2C_1, J5 SEN55, J9 E-Paper, Q1 Si1308EDL, U1 ESP32-C6-MINI-1/U, U2 SCD41-D-R2, U3 BMP280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

Commit message: Added FAN output
Parts:
- added C30: 4.7uF, Capacitor_SMD:C_0805_2012Metric, symbol Device:C
- added D1: D, Diode_SMD:D_0603_1608Metric, symbol Device:D
- added J6: FAN, Connector_JST:JST_PH_B2B-PH-K_1x02_P2.00mm_Vertical, symbol Connector:Conn_01x02_Pin
Connections:
- net +5V: now also C30.1, D1.1 (K), J6.2 (Pin_2)
- net GND: now also C30.2, D1.2 (A), J6.1 (Pin_1)
